File: OpenVideoModulator.kicad_pcb (KiCad board)
At the start: 2 copper layers, 38.6 x 24.9 mm, 22 parts, among them J1 CONN_6, J2 S-Video+Composite_Combo, P1 OSHW_LOGO, U1 AD724, Y1 4.433619M

Commit message: Ground S-Video connector shielding... AND READY FOR V1!
Changed lines of the file:
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@@
     (46 B.CrtYd user hide)
     (47 F.CrtYd user hide)
-    (49 F.Fab user hide)
+    (49 F.Fab user)
   )
   (setup
@@
     (visible_elements FFFFFF7F)
     (pcbplotparams
-      (layerselection 0x010fc_ffffffff)
+      (layerselection 0x010f0_ffffffff)
       (usegerberextensions false)
       (usegerberattributes false)
@@
       (linewidth 0.100000)
       (plotframeref false)
-      (viasonmask false)
+      (viasonmask true)
       (mode 1)
       (useauxorigin false)
@@
       (outputformat 1)
       (mirror false)
-      (drillshape 1)
+      (drillshape 0)
       (scaleselection 1)
-      (outputdirectory ""))
+      (outputdirectory "gerbers"))
   )
   (net 0 "")
@@
     (add_net GND)
     (add_net VAA)
+  )
+  (module OpenVideoModulator:AV-MDC-401 (layer F.Cu)
+    (at 153.289 66.548 90)
+    (fp_text reference J2 (at 8.05 9.15 90) (layer F.SilkS)
+      (effects (font (size 1 1) (thickness 0.15)))
+    )
+    (fp_text value S-Video+Composite_Combo (at 7.75 -16.65 90) (layer F.Fab) hide
+      (effects (font (size 1 1) (thickness 0.15)))
+    )
+    (fp_line (start 13.35 1.2) (end 13.35 0) (layer F.SilkS) (width 0.15))
+    (fp_line (start 1.65 1.2) (end 1.65 0) (layer F.SilkS) (width 0.15))
+    (fp_line (start 1.65 1.2) (end 13.35 1.2) (layer F.SilkS) (width 0.15))
+    (fp_line (start 11.65 8.1) (end 11.65 0) (layer F.SilkS) (width 0.15))
+    (fp_line (start 3.35 8.1) (end 3.35 0) (layer F.SilkS) (width 0.15))
+    (fp_line (start 3.35 8.1) (end 11.65 8.1) (layer F.SilkS) (width 0.15))
+    (fp_line (start 15 -9.8) (end 15 -15.4) (layer F.SilkS) (width 0.15))
+    (fp_line (start 0 -6.8) (end 0 0) (layer F.SilkS) (width 0.15))
+    (fp_line (start 16.05 -6.8) (end 13.55 -6.8) (layer F.SilkS) (width 0.15))
+    (fp_line (start 13.55 -9.8) (end 13.55 -6.8) (layer F.SilkS) (width 0.15))
+    (fp_line (start 13.55 -9.8) (end 16.05 -9.8) (layer F.SilkS) (width 0.15))
+    (fp_line (start 16.05 -9.8) (end 16.05 -6.8) (layer F.SilkS) (width 0.15))
+    (fp_line (start -1.05 -9.8) (end -1.05 -6.8) (layer F.SilkS) (width 0.15))
+    (fp_line (start 1.45 -6.8) (end -1.05 -6.8) (layer F.SilkS) (width 0.15))
+    (fp_line (start 1.45 -9.8) (end 1.45 -6.8) (layer F.SilkS) (width 0.15))
+    (fp_line (start -1.05 -9.8) (end 1.45 -9.8) (layer F.SilkS) (width 0.15))
+    (fp_line (start 0 -9.8) (end 0 -15.4) (layer F.SilkS) (width 0.15))
+    (fp_line (start 15 0) (end 0 0) (layer F.SilkS) (width 0.15))
+    (fp_line (start 15 -6.8) (end 15 0) (layer F.SilkS) (width 0.15))
+    (fp_line (start 0 -15.4) (end 15 -15.4) (layer F.SilkS) (width 0.15))
+    (pad "" np_thru_hole oval (at 14.8 -8.3 90) (size 2.5 3) (drill oval 2.5 3) (layers *.Cu *.Mask))
+    (pad "" np_thru_hole oval (at 0.2 -8.3 90) (size 2.5 3) (drill oval 2.5 3) (layers *.Cu *.Mask))
+    (pad 7 thru_hole oval (at 7.5 -3.2 90) (size 3.2 1.6) (drill oval 2.5 1) (layers *.Cu *.Mask)
+      (net 2 GND))
+    (pad 6 thru_hole circle (at 7.5 -14 90) (size 2 2) (drill 1.5) (layers *.Cu *.Mask)
+      (net 20 "Net-(J2-Pad6)"))
+    (pad 5 thru_hole circle (at 12.5 -14 90) (size 2 2) (drill 1.5) (layers *.Cu *.Mask)
+      (net 2 GND))
+    (pad 4 thru_hole circle (at 4.25 -9.5 90) (size 2 2) (drill 1.2) (layers *.Cu *.Mask)
+      (net 19 "Net-(J2-Pad4)"))
+    (pad 3 thru_hole circle (at 10.75 -9.5 90) (size 2 2) (drill 1.4) (layers *.Cu *.Mask)
+      (net 18 "Net-(J2-Pad3)"))
+    (pad 2 thru_hole circle (at 4.25 -7 90) (size 2 2) (drill 1.4) (layers *.Cu *.Mask)
+      (net 2 GND))
+    (pad 1 thru_hole circle (at 10.75 -7 90) (size 2 2) (drill 1.4) (layers *.Cu *.Mask)
+      (net 2 GND))
+    (model ${P3D_WALTER}/conn_av/minidin-8.wrl
+      (offset (xyz 7.5 8 0))
+      (scale (xyz 1 1.1 1.5))
+      (rotate (xyz 0 0 0))
+    )
   )
   (module Capacitor_SMD:C_0805_2012Metric_Pad1.15x1.40mm_HandSolder (layer B.Cu)
@@
     )
   )
-  (module OpenVideoModulator:AV-MDC-401 (layer F.Cu)
-    (at 153.289 66.548 90)
-    (fp_text reference J2 (at 8.05 9.15 90) (layer F.SilkS)
-      (effects (font (size 1 1) (thickness 0.15)))
-    )
-    (fp_text value S-Video+Composite_Combo (at 7.75 -16.65 90) (layer F.Fab) hide
-      (effects (font (size 1 1) (thickness 0.15)))
-    )
-    (fp_line (start 0 -15.4) (end 15 -15.4) (layer F.SilkS) (width 0.15))
-    (fp_line (start 15 -6.8) (end 15 0) (layer F.SilkS) (width 0.15))
-    (fp_line (start 15 0) (end 0 0) (layer F.SilkS) (width 0.15))
-    (fp_line (start 0 -9.8) (end 0 -15.4) (layer F.SilkS) (width 0.15))
-    (fp_line (start -1.05 -9.8) (end 1.45 -9.8) (layer F.SilkS) (width 0.15))
-    (fp_line (start 1.45 -9.8) (end 1.45 -6.8) (layer F.SilkS) (width 0.15))
-    (fp_line (start 1.45 -6.8) (end -1.05 -6.8) (layer F.SilkS) (width 0.15))
-    (fp_line (start -1.05 -9.8) (end -1.05 -6.8) (layer F.SilkS) (width 0.15))
-    (fp_line (start 16.05 -9.8) (end 16.05 -6.8) (layer F.SilkS) (width 0.15))
-    (fp_line (start 13.55 -9.8) (end 16.05 -9.8) (layer F.SilkS) (width 0.15))
-    (fp_line (start 13.55 -9.8) (end 13.55 -6.8) (layer F.SilkS) (width 0.15))
-    (fp_line (start 16.05 -6.8) (end 13.55 -6.8) (layer F.SilkS) (width 0.15))
-    (fp_line (start 0 -6.8) (end 0 0) (layer F.SilkS) (width 0.15))
-    (fp_line (start 15 -9.8) (end 15 -15.4) (layer F.SilkS) (width 0.15))
-    (fp_line (start 3.35 8.1) (end 11.65 8.1) (layer F.SilkS) (width 0.15))
-    (fp_line (start 3.35 8.1) (end 3.35 0) (layer F.SilkS) (width 0.15))
-    (fp_line (start 11.65 8.1) (end 11.65 0) (layer F.SilkS) (width 0.15))
-    (fp_line (start 1.65 1.2) (end 13.35 1.2) (layer F.SilkS) (width 0.15))
-    (fp_line (start 1.65 1.2) (end 1.65 0) (layer F.SilkS) (width 0.15))
-    (fp_line (start 13.35 1.2) (end 13.35 0) (layer F.SilkS) (width 0.15))
-    (pad 1 thru_hole circle (at 10.75 -7 90) (size 2 2) (drill 1.4) (layers *.Cu *.Mask)
-      (net 2 GND))
-    (pad 2 thru_hole circle (at 4.25 -7 90) (size 2 2) (drill 1.4) (layers *.Cu *.Mask)
-      (net 2 GND))
-    (pad 3 thru_hole circle (at 10.75 -9.5 90) (size 2 2) (drill 1.4) (layers *.Cu *.Mask)
-      (net 18 "Net-(J2-Pad3)"))
-    (pad 4 thru_hole circle (at 4.25 -9.5 90) (size 2 2) (drill 1.2) (layers *.Cu *.Mask)
-      (net 19 "Net-(J2-Pad4)"))
-    (pad 5 thru_hole circle (at 12.5 -14 90) (size 2 2) (drill 1.5) (layers *.Cu *.Mask)
-      (net 2 GND))
-    (pad 6 thru_hole circle (at 7.5 -14 90) (size 2 2) (drill 1.5) (layers *.Cu *.Mask)
-      (net 20 "Net-(J2-Pad6)"))
-    (pad "" np_thru_hole oval (at 7.5 -3.2 90) (size 3.2 1.6) (drill oval 2.5 1) (layers *.Cu *.Mask))
-    (pad "" np_thru_hole oval (at 0.2 -8.3 90) (size 2.5 3) (drill oval 2.5 3) (layers *.Cu *.Mask))
-    (pad "" np_thru_hole oval (at 14.8 -8.3 90) (size 2.5 3) (drill oval 2.5 3) (layers *.Cu *.Mask))
-    (model ${P3D_WALTER}/conn_av/minidin-8.wrl
-      (offset (xyz 7.5 8 0))
-      (scale (xyz 1 1.1 1.5))
-      (rotate (xyz 0 0 0))
-    )
-  )
   (module Crystal:Crystal_HC49-4H_Vertical (layer F.Cu)
     (at 129.4 52.832 180)
@@
     (effects (font (size 1 1) (thickness 0.2)) (justify mirror))
   )
-  (dimension 24.13 (width 0.3) (layer F.Fab)
-    (gr_text "24,130 mm" (at 108.39 62.103 90) (layer F.Fab)
+  (dimension 24.828581 (width 0.3) (layer F.Fab)
+    (gr_text "24,829 mm" (at 108.358269 62.022216 -89.8534638) (layer F.Fab)
       (effects (font (size 1.5 1.5) (thickness 0.3)))
     )
-    (feature1 (pts (xy 114.046 50.038) (xy 109.903579 50.038)))
-    (feature2 (pts (xy 114.046 74.168) (xy 109.903579 74.168)))
-    (crossbar (pts (xy 110.49 74.168) (xy 110.49 50.038)))
-    (arrow1a (pts (xy 110.49 50.038) (xy 111.076421 51.164504)))
-    (arrow1b (pts (xy 110.49 50.038) (xy 109.903579 51.164504)))
-    (arrow2a (pts (xy 110.49 74.168) (xy 111.076421 73.041496)))
-    (arrow2b (pts (xy 110.49 74.168) (xy 109.903579 73.041496)))
+    (feature1 (pts (xy 113.9825 49.5935) (xy 109.840093 49.604094)))
+    (feature2 (pts (xy 114.046 74.422) (xy 109.903593 74.432594)))
+    (crossbar (pts (xy 110.490012 74.431095) (xy 110.426512 49.602595)))
+    (arrow1a (pts (xy 110.426512 49.602595) (xy 111.015812 50.727595)))
+    (arrow1b (pts (xy 110.426512 49.602595) (xy 109.842974 50.730595)))
+    (arrow2a (pts (xy 110.490012 74.431095) (xy 111.07355 73.303095)))
+    (arrow2b (pts (xy 110.490012 74.431095) (xy 109.900712 73.306095)))
   )
   (dimension 38.608 (width 0.3) (layer F.Fab)
-    (gr_text "38,608 mm" (at 133.35 80.84) (layer F.Fab)
+    (gr_text "38,608 mm" (at 133.35 81.094) (layer F.Fab)
       (effects (font (size 1.5 1.5) (thickness 0.3)))
     )
-    (feature1 (pts (xy 152.654 74.168) (xy 152.654 79.326421)))
-    (feature2 (pts (xy 114.046 74.168) (xy 114.046 79.326421)))
-    (crossbar (pts (xy 114.046 78.74) (xy 152.654 78.74)))
-    (arrow1a (pts (xy 152.654 78.74) (xy 151.527496 79.326421)))
-    (arrow1b (pts (xy 152.654 78.74) (xy 151.527496 78.153579)))
-    (arrow2a (pts (xy 114.046 78.74) (xy 115.172504 79.326421)))
-    (arrow2b (pts (xy 114.046 78.74) (xy 115.172504 78.153579)))
+    (feature1 (pts (xy 152.654 74.422) (xy 152.654 79.580421)))
+    (feature2 (pts (xy 114.046 74.422) (xy 114.046 79.580421)))
+    (crossbar (pts (xy 114.046 78.994) (xy 152.654 78.994)))
+    (arrow1a (pts (xy 152.654 78.994) (xy 151.527496 79.580421)))
+    (arrow1b (pts (xy 152.654 78.994) (xy 151.527496 78.407579)))
+    (arrow2a (pts (xy 114.046 78.994) (xy 115.172504 79.580421)))
+    (arrow2b (pts (xy 114.046 78.994) (xy 115.172504 78.407579)))
   )
   (gr_arc (start 115.316 50.8) (end 115.316 49.53) (angle -90) (layer Edge.Cuts) (width 0.15))

Commit message: Final touches for release
Routing:
- net GND: vias 27 -> 26
Other:
- outline, holes or cut-outs redrawn
Changed lines of the file:
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@@
-(kicad_pcb (version 20171130) (host pcbnew 5.0.2)
+(kicad_pcb (version 20171130) (host pcbnew 5.1.5)
   (general
     (thickness 1.6)
     (drawings 21)
-    (tracks 154)
+    (tracks 155)
     (zones 0)
     (modules 22)
@@
     (title OpenVideoModulator)
     (date 2019-03-21)
-    (rev 1git)
+    (rev 1)
     (company SukkoPera)
     (comment 1 "Thanks to CPCWiki")
@@
     (zone_45_only yes)
     (trace_min 0.2)
-    (segment_width 0.2)
-    (edge_width 0.15)
     (via_size 0.6)
     (via_drill 0.4)
@@
     (uvia_min_size 0.2)
     (uvia_min_drill 0.1)
+    (edge_width 0.15)
+    (segment_width 0.2)
     (pcb_text_width 0.3)
     (pcb_text_size 1.5 1.5)
@@
     (descr "Through hole straight pin header, 1x06, 2.54mm pitch, single row")
     (tags "Through hole pin header THT 1x06 2.54mm single row")
-    (fp_text reference J1 (at 0 15.056) (layer F.SilkS) hide
+    (fp_text reference J1 (at 0 15.4305) (layer F.SilkS)
       (effects (font (size 1 1) (thickness 0.15)))
     )
@@
     (pad 6 thru_hole oval (at 0 12.7) (size 1.7 1.7) (drill 1) (layers *.Cu *.Mask)
       (net 7 /blue_in))
-    (model ${KISYS3DMOD}/Connector_PinHeader_2.54mm.3dshapes/PinHeader_1x06_P2.54mm_Vertical.wrl
-      (at (xyz 0 0 0))
-      (scale (xyz 1 1 1))
-      (rotate (xyz 0 0 0))
+    (model ${KISYS3DMOD}/Connector_PinHeader_2.54mm.3dshapes/PinHeader_1x06_P2.54mm_Horizontal.wrl
+      (offset (xyz 0 -12.7 0))
+      (scale (xyz 1 1 1))
+      (rotate (xyz 0 0 180))
     )
   )
@@
     (tags "resistor handsolder")
     (attr smd)
-    (fp_text reference R1 (at -2.794 0) (layer B.SilkS)
+    (fp_text reference R1 (at -2.794 0.2015) (layer B.SilkS)
       (effects (font (size 1 1) (thickness 0.15)) (justify mirror))
     )
@@
     (descr "Crystal THT HC-49-4H http://5hertz.com/pdfs/04404_D.pdf")
     (tags "THT crystalHC-49-4H")
-    (fp_text reference Y1 (at -4.331 1.651 180) (layer F.SilkS)
+    (fp_text reference Y1 (at -4.077 1.3335 180) (layer F.SilkS)
       (effects (font (size 1 1) (thickness 0.15)))
     )
@@
     (effects (font (size 1 1) (thickness 0.2)))
   )
-  (gr_text +5V (at 118.999 52.197) (layer F.SilkS)
+  (gr_text +5V (at 118.999 52.07) (layer F.SilkS)
     (effects (font (size 1 1) (thickness 0.2)))
   )
-  (gr_text NTSC (at 121.158 57.658 90) (layer F.SilkS)
+  (gr_text NTSC (at 121.158 57.785 90) (layer F.SilkS)
     (effects (font (size 0.8 0.8) (thickness 0.15)))
   )
@@
   (gr_arc (start 151.384 73.152) (end 151.384 74.422) (angle -90) (layer Edge.Cuts) (width 0.15))
   (gr_arc (start 151.384 50.8) (end 152.654 50.8) (angle -90) (layer Edge.Cuts) (width 0.15))
-  (gr_text PAL (at 121.158 64.897 90) (layer F.SilkS)
+  (gr_text PAL (at 121.158 64.77 90) (layer F.SilkS)
     (effects (font (size 0.8 0.8) (thickness 0.15)))
   )
   (gr_line (start 114.046 73.152) (end 114.046 50.8) (layer Edge.Cuts) (width 0.15))
-  (gr_line (start 151.4 74.422) (end 115.316 74.422) (layer Edge.Cuts) (width 0.15))
+  (gr_line (start 151.384 74.422) (end 115.316 74.422) (layer Edge.Cuts) (width 0.15))
   (gr_line (start 152.654 50.8) (end 152.654 73.152) (layer Edge.Cuts) (width 0.15))
-  (gr_line (start 115.316 49.53) (end 151.4 49.53) (layer Edge.Cuts) (width 0.15))
+  (gr_line (start 115.316 49.53) (end 151.384 49.53) (layer Edge.Cuts) (width 0.15))
   (segment (start 124.406 52.832) (end 124.66 53.086) (width 0.25) (layer B.Cu) (net 1) (status 30))
   (segment (start 122.437 52.832) (end 124.52 52.832) (width 0.25) (layer B.Cu) (net 1) (status 30))
@@
   (segment (start 121.2215 62.768) (end 123.8915 62.768) (width 0.25) (layer F.Cu) (net 2))
   (via (at 114.935 73.533) (size 0.8) (drill 0.6) (layers F.Cu B.Cu) (net 2))
-  (via (at 124.11075 73.533) (size 0.8) (drill 0.6) (layers F.Cu B.Cu) (net 2))
-  (via (at 133.2865 73.533) (size 0.8) (drill 0.6) (layers F.Cu B.Cu) (net 2))
+  (via (at 132.334 73.533) (size 0.8) (drill 0.6) (layers F.Cu B.Cu) (net 2))
   (via (at 142.46225 73.533) (size 0.8) (drill 0.6) (layers F.Cu B.Cu) (net 2))
   (via (at 151.638 73.533) (size 0.8) (drill 0.6) (layers F.Cu B.Cu) (net 2))
   (via (at 151.638 50.292) (size 0.8) (drill 0.6) (layers F.Cu B.Cu) (net 2))
   (via (at 114.935 50.292) (size 0.8) (drill 0.6) (layers F.Cu B.Cu) (net 2))
-  (via (at 124.11075 50.292) (size 0.8) (drill 0.6) (layers F.Cu B.Cu) (net 2))
+  (via (at 121.7295 50.292) (size 0.8) (drill 0.6) (layers F.Cu B.Cu) (net 2))
   (via (at 133.2865 50.292) (size 0.8) (drill 0.6) (layers F.Cu B.Cu) (net 2))
   (via (at 142.46225 50.292) (size 0.8) (drill 0.6) (layers F.Cu B.Cu) (net 2))
   (via (at 114.935 68.453) (size 0.8) (drill 0.6) (layers F.Cu B.Cu) (net 2))
   (via (at 151.638 65.616666) (size 0.8) (drill 0.6) (layers F.Cu B.Cu) (net 2))
-  (via (at 151.638 57.954333) (size 0.8) (drill 0.6) (layers F.Cu B.Cu) (net 2))
   (via (at 122.428 68.834) (size 0.8) (drill 0.6) (layers F.Cu B.Cu) (net 2))
-  (via (at 129.286 69.215) (size 0.8) (drill 0.6) (layers F.Cu B.Cu) (net 2))
+  (via (at 128.9685 69.215) (size 0.8) (drill 0.6) (layers F.Cu B.Cu) (net 2))
   (via (at 136.652 69.215) (size 0.8) (drill 0.6) (layers F.Cu B.Cu) (net 2))
-  (via (at 117.983 62.23) (size 0.8) (drill 0.6) (layers F.Cu B.Cu) (net 2))
+  (via (at 118.745 60.959999) (size 0.8) (drill 0.6) (layers F.Cu B.Cu) (net 2))
   (via (at 121.412 65.278) (size 0.8) (drill 0.6) (layers F.Cu B.Cu) (net 2))
   (via (at 127.381 65.151) (size 0.8) (drill 0.6) (layers F.Cu B.Cu) (net 2))
@@
   (via (at 139.319 61.087) (size 0.8) (drill 0.6) (layers F.Cu B.Cu) (net 2))
   (via (at 139.319 56.896) (size 0.8) (drill 0.6) (layers F.Cu B.Cu) (net 2))
+  (via (at 124.11075 73.533) (size 0.8) (drill 0.6) (layers F.Cu B.Cu) (net 2))
   (segment (start 125.652 60.071) (end 124.206 60.071) (width 0.25) (layer B.Cu) (net 3) (status 10))
   (segment (start 123.825 59.69) (end 122.437 59.69) (width 0.25) (layer B.Cu) (net 3) (status 20))
@@
   (segment (start 123.825 55.626) (end 123.317 55.118) (width 0.25) (layer B.Cu) (net 5))
   (segment (start 120.387 55.118) (end 120.387 57.404) (width 0.25) (layer B.Cu) (net 6) (status 30))
-  (via (at 118.872 57.404) (size 0.6) (drill 0.4) (layers F.Cu B.Cu) (net 6))
-  (segment (start 116.078 62.23) (end 118.872 59.436) (width 0.25) (layer F.Cu) (net 6) (status 10))
-  (segment (start 118.872 59.436) (end 118.872 57.404) (width 0.25) (layer F.Cu) (net 6))
-  (segment (start 118.872 57.404) (end 120.387 57.404) (width 0.25) (layer B.Cu) (net 6) (status 20))
+  (via (at 118.872 58.54701) (size 0.6) (drill 0.4) (layers F.Cu B.Cu) (net 6))
+  (segment (start 118.872 59.436) (end 118.872 58.54701) (width 0.25) (layer F.Cu) (net 6))
+  (segment (start 116.078 62.23) (end 118.872 59.436) (width 0.25) (layer F.Cu) (net 6))
+  (segment (start 118.872 57.7215) (end 119.1895 57.404) (width 0.25) (layer B.Cu) (net 6))
+  (segment (start 118.872 58.54701) (end 118.872 57.7215) (width 0.25) (layer B.Cu) (net 6))
+  (segment (start 120.387 57.404) (end 119.1895 57.404) (width 0.25) (layer B.Cu) (net 6))
   (segment (start 120.387 64.262) (end 120.387 66.548) (width 0.25) (layer B.Cu) (net 7) (status 30))
   (segment (start 116.078 64.77) (end 117.856 66.548) (width 0.25) (layer B.Cu) (net 7) (status 10))
