File: OpenVideoModulator.kicad_pcb (KiCad board)
At the start: 2 copper layers, 35.3 x 24.9 mm, 25 parts, among them J1 CONN_6, J2 VIDEOCOMP_OUT, J3 SVIDEO_OUT, U1 AD724, Y1 4.433619M

Commit message: Rename J2
Parts:
- J2: value VIDEOCOMP_OUT -> COMPVIDEO_OUT
Changed lines of the file:
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@@
   (title_block
     (title OpenVideoModulator)
-    (date 2019-03-21)
-    (rev 1)
+    (date 2020-03-30)
+    (rev 2)
     (company SukkoPera)
     (comment 1 "Thanks to CPCWiki")
@@
       (effects (font (size 1 1) (thickness 0.15)))
     )
-    (fp_text value VIDEOCOMP_OUT (at 10.69 15.225 90) (layer F.Fab)
+    (fp_text value COMPVIDEO_OUT (at 10.69 15.225 90) (layer F.Fab)
       (effects (font (size 1 1) (thickness 0.015)))
     )
@@
   (segment (start 123.8915 60.168) (end 124.079 59.9805) (width 0.25) (layer F.Cu) (net 9) (status 30))
   (segment (start 121.2215 60.168) (end 123.8915 60.168) (width 0.25) (layer F.Cu) (net 9) (status 30))
-  (segment (start 132.08225 67.945) (end 132.9055 67.945) (width 0.25) (layer B.Cu) (net 19))
-  (segment (start 128.20875 71.8185) (end 132.08225 67.945) (width 0.25) (layer B.Cu) (net 19))
-  (segment (start 127.15875 71.8185) (end 128.20875 71.8185) (width 0.25) (layer B.Cu) (net 19) (status 10))
-  (segment (start 132.461 67.945) (end 132.9055 67.945) (width 0.25) (layer B.Cu) (net 19))
   (segment (start 133.096 67.31) (end 132.715 67.691) (width 0.25) (layer F.Cu) (net 10))
   (segment (start 132.715 67.691) (end 123.2535 67.691) (width 0.25) (layer F.Cu) (net 10))
@@
   (segment (start 134.484 64.008) (end 134.484 67.301) (width 0.25) (layer F.Cu) (net 12) (status 10))
   (segment (start 134.484 67.301) (end 135.0645 67.8815) (width 0.25) (layer F.Cu) (net 12))
-  (segment (start 121.2555 71.8185) (end 119.253 71.8185) (width 0.25) (layer B.Cu) (net 18) (status 20))
-  (segment (start 124.9766 68.0974) (end 121.2555 71.8185) (width 0.25) (layer B.Cu) (net 18))
-  (segment (start 131.2672 68.0974) (end 124.9766 68.0974) (width 0.25) (layer B.Cu) (net 18))
-  (segment (start 136.652 66.929) (end 136.144 67.437) (width 0.25) (layer B.Cu) (net 18))
-  (segment (start 136.144 67.437) (end 131.9276 67.437) (width 0.25) (layer B.Cu) (net 18))
-  (segment (start 131.9276 67.437) (end 131.2672 68.0974) (width 0.25) (layer B.Cu) (net 18))
-  (segment (start 134.952 57.531) (end 136.906 57.531) (width 0.25) (layer B.Cu) (net 20) (status 10))
-  (segment (start 136.906 57.531) (end 137.668 58.293) (width 0.25) (layer B.Cu) (net 20))
-  (segment (start 137.668 58.293) (end 137.668 66.929) (width 0.25) (layer B.Cu) (net 20))
-  (segment (start 135.0645 71.8185) (end 137.16 71.8185) (width 0.25) (layer B.Cu) (net 20) (status 10))
-  (segment (start 137.668 71.3105) (end 137.668 67.056) (width 0.25) (layer B.Cu) (net 20))
-  (segment (start 137.16 71.8185) (end 137.668 71.3105) (width 0.25) (layer B.Cu) (net 20))
-  (segment (start 137.668 67.056) (end 137.668 66.929) (width 0.25) (layer B.Cu) (net 20))
   (segment (start 132.2832 66.421) (end 134.952 66.421) (width 0.25) (layer B.Cu) (net 13) (status 20))
   (segment (start 115.32501 67.57301) (end 131.13119 67.57301) (width 0.25) (layer B.Cu) (net 13))
@@
   (segment (start 138.049 66.1035) (end 139.954 68.0085) (width 0.25) (layer F.Cu) (net 17) (status 20))
   (segment (start 138.049 65.532) (end 138.049 66.1035) (width 0.25) (layer F.Cu) (net 17))
+  (segment (start 121.2555 71.8185) (end 119.253 71.8185) (width 0.25) (layer B.Cu) (net 18) (status 20))
+  (segment (start 124.9766 68.0974) (end 121.2555 71.8185) (width 0.25) (layer B.Cu) (net 18))
+  (segment (start 131.2672 68.0974) (end 124.9766 68.0974) (width 0.25) (layer B.Cu) (net 18))
+  (segment (start 136.652 66.929) (end 136.144 67.437) (width 0.25) (layer B.Cu) (net 18))
+  (segment (start 136.144 67.437) (end 131.9276 67.437) (width 0.25) (layer B.Cu) (net 18))
+  (segment (start 131.9276 67.437) (end 131.2672 68.0974) (width 0.25) (layer B.Cu) (net 18))
   (segment (start 136.652 60.452) (end 136.652 60.833) (width 0.25) (layer B.Cu) (net 18))
   (segment (start 136.652 60.833) (end 136.652 66.929) (width 0.25) (layer B.Cu) (net 18))
@@
   (segment (start 136.271 58.801) (end 136.652 59.182) (width 0.25) (layer B.Cu) (net 18))
   (segment (start 134.952 58.801) (end 136.271 58.801) (width 0.25) (layer B.Cu) (net 18) (status 10))
+  (segment (start 132.08225 67.945) (end 132.9055 67.945) (width 0.25) (layer B.Cu) (net 19))
+  (segment (start 128.20875 71.8185) (end 132.08225 67.945) (width 0.25) (layer B.Cu) (net 19))
+  (segment (start 127.15875 71.8185) (end 128.20875 71.8185) (width 0.25) (layer B.Cu) (net 19) (status 10))
+  (segment (start 132.461 67.945) (end 132.9055 67.945) (width 0.25) (layer B.Cu) (net 19))
   (segment (start 136.398 67.945) (end 137.16 67.183) (width 0.25) (layer B.Cu) (net 19))
   (segment (start 132.9055 67.945) (end 136.398 67.945) (width 0.25) (layer B.Cu) (net 19))
@@
   (segment (start 133.985 60.071) (end 134.952 60.071) (width 0.25) (layer B.Cu) (net 19) (status 20))
   (segment (start 133.604 58.513998) (end 133.604 59.69) (width 0.25) (layer B.Cu) (net 19))
+  (segment (start 134.952 57.531) (end 136.906 57.531) (width 0.25) (layer B.Cu) (net 20) (status 10))
+  (segment (start 136.906 57.531) (end 137.668 58.293) (width 0.25) (layer B.Cu) (net 20))
+  (segment (start 137.668 58.293) (end 137.668 66.929) (width 0.25) (layer B.Cu) (net 20))
+  (segment (start 135.0645 71.8185) (end 137.16 71.8185) (width 0.25) (layer B.Cu) (net 20) (status 10))
+  (segment (start 137.668 71.3105) (end 137.668 67.056) (width 0.25) (layer B.Cu) (net 20))
+  (segment (start 137.16 71.8185) (end 137.668 71.3105) (width 0.25) (layer B.Cu) (net 20))
+  (segment (start 137.668 67.056) (end 137.668 66.929) (width 0.25) (layer B.Cu) (net 20))
   (zone (net 2) (net_name GND) (layer B.Cu) (hatch edge 0.508)
     (connect_pads (clearance 0.1))
