File: OpenVideoModulator.sch (KiCad schematic (older format))
At the start: 25 parts, among them J1 CONN_6, J2 COMPVIDEO_OUT, J3 SVIDEO_OUT, U1 AD724, Y1 4.433619M

Commit message: Done
Parts:
- J2: footprint (none) -> OpenVideoModulator:Pin_Header_Straight_1x02-ModSilkS
- J3: footprint (none) -> OpenVideoModulator:MiniDIN4
Changed lines of the file:
@@
 F 0 "J3" H 9365 4875 50  0000 C CNN
 F 1 "SVIDEO_OUT" H 9365 4775 50  0000 C CNN
-F 2 "" H 9365 4390 50  0001 C CNN
+F 2 "OpenVideoModulator:MiniDIN4" H 9365 4390 50  0001 C CNN
 F 3 "http://service.powerdynamics.com/ec/Catalog17/Section%2011.pdf" H 9365 4390 50  0001 C CNN
 	1    9365 4390
@@
 F 0 "J2" H 9117 3409 50  0000 R CNN
 F 1 "COMPVIDEO_OUT" H 9117 3318 50  0000 R CNN
-F 2 "" H 9145 3435 50  0001 C CNN
+F 2 "OpenVideoModulator:Pin_Header_Straight_1x02-ModSilkS" H 9145 3435 50  0001 C CNN
 F 3 "~" H 9145 3435 50  0001 C CNN
 	1    9145 3435
